Commit message: new transformation between world and robot, and between wrist and hand, as provided by innsbruck

File: ros_pkgs/hardware/torso_uibk/urdf/table.xacro (robot description, xacro)
@@ -1,79 +1,59 @@
 <?xml version="1.0"?>
 <robot xmlns:xacro="http://www.ros.org/wiki/xacro">
-  <macro name="model_table" params="parent name *origin">
-    <joint name="${parent}_${name}_base_joint" type="fixed">
-      <insert_block name="origin"/>
-      <parent link="${parent}_link"/>
-      <child link="${name}_link"/>
+<property name="leg_width" value="0.03" />
+<property name="border_offset" value="0.055" />
+<macro name="table_leg" params="parent name *origin">
+    <joint name="${name}_joint" type="fixed">
+        <insert_block name="origin"/>
+        <parent link="${parent}" />
+        <child link="${name}_link" />
     </joint>
     <link name="${name}_link">
-      <visual>
-	<origin xyz="0.29 0.355 0.34"/>
-	<geometry>
-	  <box size="0.04 0.04 0.68"/>
-	</geometry>
-	<material name="LightGrey"/>
-      </visual>
-      <visual>
-	<origin xyz="-0.29 0.355 0.34"/>
-	<geometry>
-	  <box size="0.04 0.04 0.68"/>
-	</geometry>
-	<material name="DarkGrey"/>
-      </visual>
-      <visual>
-	<origin xyz="0.29 -0.355 0.34"/>
-	<geometry>
-	  <box size="0.04 0.04 0.68"/>
-	</geometry>
-	<material name="DarkGrey"/>
-      </visual>
-      <visual>
-	<origin xyz="-0.29 -0.355 0.34"/>
-	<geometry>
-	  <box size="0.04 0.04 0.68"/>
-	</geometry>
-	<material name="DarkGrey"/>
-      </visual>
-      <!-- platte -->
-      <visual>
-	<origin xyz="0 0 0.695"/>
-	<geometry>
-	  <box size="0.7 1.4 0.03"/>
-	</geometry>
-	<material name="LightGrey"/>
-      </visual>
-      <collision>
-	<origin xyz="0.29 0.355 0.34"/>
-	<geometry>
-	  <box size="0.04 0.04 0.68"/>
-	</geometry>
-      </collision>
-      <collision>
-	<origin xyz="-0.29 0.355 0.34"/>
-	<geometry>
-	  <box size="0.04 0.04 0.68"/>
-	</geometry>
-      </collision>
-      <collision>
-	<origin xyz="0.29 -0.355 0.34"/>
-	<geometry>
-	  <box size="0.04 0.04 0.68"/>
-	</geometry>
-      </collision>
-      <collision>
-	<origin xyz="-0.29 -0.355 0.34"/>
-	<geometry>
-	  <box size="0.04 0.04 0.68"/>
-	</geometry>
-      </collision>
-      <!-- platte -->
-      <collision>
-	<origin xyz="0 0 0.695"/>
-	<geometry>
-	  <box size="0.7 1.4 0.03"/>
-	</geometry>
-      </collision>
+		<visual>
+			<geometry>
+				<box size="${leg_width} -${leg_width} ${height - plate_thickness}"/>
+			</geometry>
+			<material name="Black"/>
+		</visual>
+		<collision>
+			<geometry>
+				<box size="${leg_width} -${leg_width} ${height - plate_thickness}"/>
+			</geometry>
+		</collision>
     </link>
-  </macro>
+</macro>
+<macro name="model_table" params="parent name *origin length width height plate_thickness">
+    <joint name="${parent}_${name}_base_joint" type="fixed">
+        <insert_block name="origin"/>
+        <parent link="${parent}_link"/>
+        <child link="${name}_plate_link"/>
+    </joint>
+    <link name="${name}_plate_link">
+        <visual>
+            <origin xyz="${1/2 * length} ${-1/2 * width} ${-1/2 * plate_thickness}"/>
+            <geometry>
+                <box size="${length} ${width} ${plate_thickness}"/>
+			</geometry>
+			<material name="LightGrey"/>
+		</visual>
+        <collision>
+            <origin xyz="${1/2 * length} ${-1/2 * width} ${-1/2 * plate_thickness}"/>
+            <geometry>
+                <box size="${length} ${width} ${plate_thickness}"/>
+            </geometry>
+        </collision>
+    </link>
+    <xacro:table_leg parent="${name}_plate_link" name="leg_0">
+        <origin xyz="${border_offset} -${border_offset} -${1/2 * (plate_thickness + height)}"/>
+    </xacro:table_leg>
+    <xacro:table_leg parent="${name}_plate_link" name="leg_1">
+        <origin xyz="${length - border_offset} -${border_offset} -${1/2 * (plate_thickness + height)}"/>
+    </xacro:table_leg>
+    <xacro:table_leg parent="${name}_plate_link" name="leg_2">
+        <origin xyz="${border_offset} -${width - border_offset} -${1/2 * (plate_thickness + height)}"/>
+    </xacro:table_leg>
+    <xacro:table_leg parent="${name}_plate_link" name="leg_3">
+        <origin xyz="${length - border_offset} -${width - border_offset} -${1/2 * (plate_thickness + height)}"/>
+    </xacro:table_leg>
+</macro>
 </robot>

File: ros_pkgs/hardware/torso_uibk/urdf/torso.xacro (robot description, xacro)
@@ -1,18 +1,23 @@
 <?xml version="1.0"?>
 <robot xmlns:xacro="http://www.ros.org/wiki/xacro">
-  <macro name="model_torso" params="parent name *origin">
-    <joint name="${parent}_${name}_base_joint" type="fixed">
-      <insert_block name="origin"/>
-      <parent link="${parent}_link"/>
-      <child link="${name}_link"/>
-    </joint>
-    <link name="${name}_link">
-      <visual>
-	<geometry>
-	  <mesh filename="package://torso_uibk/meshes/torso.stl"/>
-	</geometry>
-	<material name="Silver"/>
-      </visual>
-    </link>
-  </macro>
+<macro name="model_torso" params="parent name *origin">
+  <joint name="${parent}_${name}_base_joint" type="fixed">
+    <insert_block name="origin"/>
+    <parent link="${parent}_link"/>
+    <child link="${name}_link"/>
+  </joint>
+  <link name="${name}_link">
+    <visual>
+      <geometry>
+        <mesh filename="package://torso_uibk/meshes/torso.stl"/>
+      </geometry>
+      <material name="Silver"/>
+    </visual>
+    <collision>
+      <geometry>
+        <mesh filename="package://torso_uibk/meshes/torso.stl"/>
+      </geometry>
+    </collision>
+  </link>
+</macro>
 </robot>

File: ros_pkgs/hardware/uibk_robot/urdf/uibk_robot.urdf.xacro (robot description, xacro)
@@ -8,25 +8,30 @@
   <xacro:include filename="$(find schunk_description)/urdf/sdh/sdh.urdf.xacro" />
   <link name="world_link" />
-  <xacro:model_table name="table" parent="world">
-    <origin xyz="0.75 -0.0748 0"/>
+  <xacro:model_table name="table"
+                    parent="world"
+                    length="2.22"
+                    width="0.8"
+                    height="0.734"
+                    plate_thickness="0.1">
+    <origin xyz="-0.029 -0.3 0" rpy="0 0 1.5708"/>
   </xacro:model_table>
   <xacro:model_torso name="torso" parent="world">
-    <origin xyz="0 0 0"/>
+    <origin xyz="-0.4723 0.6767 -0.734"/>
   </xacro:model_torso>
-  <xacro:kuka_lwr_arm parent="torso" name="leftArm" right="1">
-    <origin xyz="-0.0199 0.0661 1.34"
-	    rpy="-1.9392 -0.3456 -0.2952"/>
+  <xacro:kuka_lwr_arm parent="world" name="left" right="-1">
+    <origin xyz="-0.4923 0.7541 0.6295"
+      rpy="1.9485 -0.2114 2.6898"/>
   </xacro:kuka_lwr_arm>
-  <xacro:kuka_lwr_arm parent="torso" name="rightArm" right="1">
-    <origin xyz="-0.0202 -0.0663 1.3401"
-	    rpy="1.9386 0.3471 0.6879"/>
+  <xacro:kuka_lwr_arm parent="world" name="right" right="1">
+    <origin xyz="-0.4962 0.5992 0.6335"
+      rpy="-2.0628 0.7628 -3.1287"/>
   </xacro:kuka_lwr_arm>
-  <xacro:schunk_sdh parent="leftArm_arm_7_link" name="leftGripper">
+  <xacro:schunk_sdh parent="left_arm_7_link" name="leftGripper">
     <origin xyz="0 0 0"
-	    rpy="0 0 0"/>
+      rpy="0 0 ${-1/2 * M_PI}"/>
   </xacro:schunk_sdh>
-  <xacro:schunk_sdh parent="rightArm_arm_7_link" name="rightGripper">
+  <xacro:schunk_sdh parent="right_arm_7_link" name="rightGripper">
     <origin xyz="0 0 0"
-	    rpy="0 0 0"/>
+      rpy="0 0 ${1/2 * M_PI}"/>
   </xacro:schunk_sdh>
 </robot>
