Commit message: demo ported to hydro, it works in simulation, need to be tested in real robot

File: ros_pkgs/hardware/lwr/lwr_description/urdf/kuka_lwr_arm.urdf.xacro (robot description, xacro)
@@ -1,6 +1,6 @@
 <?xml version="1.0"?>
-<robot name="lwr">
-  <include filename="kuka_lwr_arm_defs.xacro"/>
-  <include filename="materials.urdf"/>
+<robot name="lwr" xmlns:xacro="http://www.ros.org/wiki/xacro" >
+  <xacro:include filename="kuka_lwr_arm_defs.xacro"/>
+  <xacro:include filename="materials.urdf"/>
   <link name="world_link">
     <inertial>
@@ -24,6 +24,6 @@
     </collision>
   </link>
-  <kuka_lwr_arm parent="world" name="lwr" right="1">
+  <xacro:kuka_lwr_arm parent="world" name="lwr" right="1">
     <origin xyz="0 0 1.0" rpy="0 0 0"/>
-  </kuka_lwr_arm>
+  </xacro:kuka_lwr_arm>
 </robot>

File: ros_pkgs/hardware/lwr/lwr_description/urdf/kuka_lwr_arm_defs.xacro (robot description, xacro)
@@ -2,13 +2,14 @@
 <robot xmlns:sensor="http://playerstage.sourceforge.net/gazebo/xmlschema/#sensor"
        xmlns:controller="http://playerstage.sourceforge.net/gazebo/xmlschema/#controller"
-       xmlns:interface="http://playerstage.sourceforge.net/gazebo/xmlschema/#interface">
-  <include filename="$(find lwr_description)/urdf/util_defs.xacro"/>
-  <property name="arm_elem_base_mass" value="2.0"/>
-  <property name="arm_elem_link_mass" value="2.0"/>
-  <property name="arm_elem_end_link_mass" value="2.0"/>
-  <property name="arm_elem_ball_link_mass" value="2.0"/>
-  <property name="arm_velocity_scale_factor" value="1"/>
+       xmlns:interface="http://playerstage.sourceforge.net/gazebo/xmlschema/#interface"
+       xmlns:xacro="http://www.ros.org/wiki/xacro">
+  <xacro:include filename="$(find lwr_description)/urdf/util_defs.xacro"/>
+  <xacro:property name="arm_elem_base_mass" value="2.0"/>
+  <xacro:property name="arm_elem_link_mass" value="2.0"/>
+  <xacro:property name="arm_elem_end_link_mass" value="2.0"/>
+  <xacro:property name="arm_elem_ball_link_mass" value="2.0"/>
+  <xacro:property name="arm_velocity_scale_factor" value="0.1"/>
   <!-- right is either 1 (for right arm) or -1 (for left arm) -->
-  <macro name="kuka_lwr_arm" params="parent name right *origin">
+  <xacro:macro name="kuka_lwr_arm" params="parent name right *origin">
     <!-- First (shoulder) element of the arm. Fixed to its parent. -->
     <joint name="${parent}_${name}_arm_base_joint" type="fixed">
@@ -17,5 +18,15 @@
       <child link="calib_${name}_arm_base_link"/>
     </joint>
-    <link name="calib_${name}_arm_base_link">
+    <!-- In the original setting the arm was rotated around 180° around the z axis because
+         the point at the arm base, where the cables are located should point to the direction
+	 of the positive x axis of the arm reference frame. This link is used to correct that -->
+    <link name="calib_${name}_arm_base_link" />
+    <!-- Rotate arm around 180° along z axis -->
+    <joint name="calib_${name}_arm_base_joint" type="fixed">
+      <origin xyz="0 0 0" rpy="0 0 ${M_PI}" />
+      <parent link="calib_${name}_arm_base_link" />
+      <child link="${name}_arm_base_link" />
+    </joint>
+    <link name="${name}_arm_base_link">
       <inertial>
         <mass value="${arm_elem_base_mass}"/>
@@ -55,5 +66,5 @@
                          k_velocity="30"/>
       <dynamics damping="1.0"/>
-      <parent link="calib_${name}_arm_base_link"/>
+      <parent link="${name}_arm_base_link"/>
       <child link="${name}_arm_1_link"/>
     </joint>
@@ -443,4 +454,4 @@
       <mechanicalReduction>1.0</mechanicalReduction>
     </transmission>
-  </macro>
+  </xacro:macro>
 </robot>

File: ros_pkgs/hardware/lwr/lwr_description/urdf/util_defs.xacro (robot description, xacro)
@@ -1,23 +1,25 @@
 <?xml version="1.0"?>
-<robot xmlns:sensor="http://playerstage.sourceforge.net/gazebo/xmlschema/#sensor"
+<!--robot xmlns:sensor="http://playerstage.sourceforge.net/gazebo/xmlschema/#sensor"
        xmlns:controller="http://playerstage.sourceforge.net/gazebo/xmlschema/#controller"
-       xmlns:interface="http://playerstage.sourceforge.net/gazebo/xmlschema/#interface">
-  <property name="M_PI" value="3.1415926535897931" />
+       xmlns:interface="http://playerstage.sourceforge.net/gazebo/xmlschema/#interface"
+       xmlns:xacro="http://ros.org/wiki/xacro"-->
+<robot xmlns:xacro="http://ros.org/wiki/xacro">
+  <xacro:property name="M_PI" value="3.1415926535897931" />
   <!--
      Little helper macro to define the inertia matrix needed
      for links.
      -->
-  <macro name="cuboid_inertia_def" params="width height length mass">
+  <xacro:macro name="cuboid_inertia_def" params="width height length mass">
     <inertia ixx="${mass * (height * height + length * length) / 12)}"
              iyy="${mass * (width * width + length * length) / 12)}"
              izz="${mass * (width * width + height * height) / 12)}"
              ixy="0" iyz="0" ixz="0"/>
-  </macro>
+  </xacro:macro>
   <!-- length is along the y-axis! -->
-  <macro name="cylinder_inertia_def" params="radius length mass">
+  <xacro:macro name="cylinder_inertia_def" params="radius length mass">
     <inertia ixx="${mass * (3 * radius * radius + length * length) / 12)}"
              iyy="${mass * radius* radius / 2)}"
              izz="${mass * (3 * radius * radius + length * length) / 12)}"
              ixy="0" iyz="0" ixz="0"/>
-  </macro>
+  </xacro:macro>
 </robot>

File: ros_pkgs/hardware/sdh/schunk_description/urdf/sdh/sdh.urdf.xacro (robot description, xacro)
@@ -4,7 +4,7 @@
        xmlns:interface="http://playerstage.sourceforge.net/gazebo/xmlschema/#interface"
        xmlns:xacro="http://ros.org/wiki/xacro">
-	<include filename="$(find schunk_description)/urdf/sdh/sdh.gazebo.xacro" />
-	<include filename="$(find schunk_description)/urdf/sdh/sdh.transmission.xacro" />
-	<include filename="$(find schunk_description)/urdf/materials.urdf.xacro" />
+	<xacro:include filename="$(find schunk_description)/urdf/sdh/sdh.gazebo.xacro" />
+	<xacro:include filename="$(find schunk_description)/urdf/sdh/sdh.transmission.xacro" />
+	<xacro:include filename="$(find schunk_description)/urdf/materials.urdf.xacro" />
 	<xacro:macro name="schunk_sdh" params="parent name *origin">
 		<!-- joint between arm_7_link and sdh_palm_link -->

File: ros_pkgs/hardware/torso_uibk/urdf/table.xacro (robot description, xacro)
@@ -1,7 +1,7 @@
 <?xml version="1.0"?>
 <robot xmlns:xacro="http://www.ros.org/wiki/xacro">
-<property name="leg_width" value="0.03" />
-<property name="border_offset" value="0.055" />
-<macro name="table_leg" params="parent name *origin">
+<xacro:property name="leg_width" value="0.03" />
+<xacro:property name="border_offset" value="0.055" />
+<xacro:macro name="table_leg" params="parent name *origin">
     <joint name="${name}_joint" type="fixed">
         <insert_block name="origin"/>
@@ -22,6 +22,6 @@
 		</collision>
     </link>
-</macro>
-<macro name="model_table" params="parent name *origin length width height plate_thickness">
+</xacro:macro>
+<xacro:macro name="model_table" params="parent name *origin length width height plate_thickness">
     <joint name="${parent}_${name}_base_joint" type="fixed">
         <insert_block name="origin"/>
@@ -56,4 +56,4 @@
         <origin xyz="${length - border_offset} -${width - border_offset} -${1/2 * (plate_thickness + height)}"/>
     </xacro:table_leg>
-</macro>
+</xacro:macro>
 </robot>

File: ros_pkgs/hardware/torso_uibk/urdf/torso.xacro (robot description, xacro)
@@ -1,5 +1,5 @@
 <?xml version="1.0"?>
 <robot xmlns:xacro="http://www.ros.org/wiki/xacro">
-<macro name="model_torso" params="parent name *origin">
+<xacro:macro name="model_torso" params="parent name *origin">
   <joint name="${parent}_${name}_base_joint" type="fixed">
     <insert_block name="origin"/>
@@ -20,4 +20,4 @@
     </collision>
   </link>
-</macro>
+</xacro:macro>
 </robot>

File: ros_pkgs/hardware/uibk_robot/urdf/uibk_robot.urdf.xacro (robot description, xacro)
@@ -9,10 +9,10 @@
   <link name="world_link" />
   <xacro:model_table name="table"
-                    parent="world"
-                    length="2.22"
-                    width="0.8"
-                    height="0.734"
-                    plate_thickness="0.1">
-    <origin xyz="-0.029 -0.3 0" rpy="0 0 1.5708"/>
+         parent="world"
+         length="2.22"
+         width="1.2"
+         height="0.8"
+         plate_thickness="0.11">
+    <origin xyz="-0.42 -0.3 0.08" rpy="0 0 1.5708"/>
   </xacro:model_table>
   <xacro:model_torso name="torso" parent="world">
@@ -27,11 +27,91 @@
       rpy="-2.0628 0.7628 -3.1287"/>
   </xacro:kuka_lwr_arm>
-  <xacro:schunk_sdh parent="left_arm_7_link" name="leftGripper">
-    <origin xyz="0 0 0"
-      rpy="0 0 ${-1/2 * M_PI}"/>
+  <!-- joint between arm_7_link and the connector ring -->
+  <joint name="left_sdh_connector_joint" type="fixed" >
+    <origin xyz="0 0 0" />
+    <parent link="left_arm_7_link" />
+    <child link="left_sdh_connector_link" />
+  </joint>
+  <!-- connector ring added to adjust distance to arm connector -->
+  <link name="left_sdh_connector_link">
+    <visual>
+      <origin xyz="0 0 0.0084" rpy="0 0 0" />
+      <geometry>
+        <cylinder radius="0.02735" length="0.0168" />
+      </geometry>
+      <material name="DarkGrey" />
+    </visual>
+    <collision>
+      <origin xyz="0 0 0.0084" rpy="0 0 0" />
+      <geometry>
+        <cylinder radius="0.02735" length="0.0168" />
+      </geometry>
+    </collision>
+  </link>
+  <xacro:schunk_sdh parent="left_sdh_connector_link" name="left_sdh">
+    <origin xyz="0 0 0.0168" rpy="0 0 ${-1/2 * M_PI}"/>
   </xacro:schunk_sdh>
-  <xacro:schunk_sdh parent="right_arm_7_link" name="rightGripper">
-    <origin xyz="0 0 0"
-      rpy="0 0 ${1/2 * M_PI}"/>
+  <!-- This connector can be a macro inside the hand package descrption -->
+  <!-- joint between arm_7_link and the connector ring -->
+  <joint name="right_sdh_connector_joint" type="fixed" >
+    <origin xyz="0 0 0" />
+      <parent link="right_arm_7_link" />
+    <child link="right_sdh_connector_link" />
+  </joint>
+<!-- connector ring added to adjust distance to arm connector -->
+  <link name="right_sdh_connector_link">
+    <visual>
+      <origin xyz="0 0 0.0084" rpy="0 0 0" />
+      <geometry>
+        <cylinder radius="0.02735" length="0.0168" />
+      </geometry>
+      <material name="DarkGrey" />
+    </visual>
+    <collision>
+      <origin xyz="0 0 0.0084" rpy="0 0 0" />
+      <geometry>
+        <cylinder radius="0.02735" length="0.0168" />
+      </geometry>
+    </collision>
+  </link>
+  <xacro:schunk_sdh parent="right_sdh_connector_link" name="right_sdh">
+    <origin xyz="0 0 0.0168" rpy="0 0 ${1/2 * M_PI}"/>
   </xacro:schunk_sdh>
+  <!-- HEAD -->
+    <!-- joint between arm_7_link and the connector ring -->
+  <joint name="world_to_kit_head" type="fixed" >
+    <origin xyz="-0.35 0.675 0.85" rpy="0 0 0" />
+    <parent link="world_link" />
+    <child link="kit_head_link" />
+  </joint>
+  <link name="kit_head_link">
+    <visual>
+      <origin xyz="0 0 0" rpy="0 0 0" />
+      <geometry>
+        <cylinder radius="0.15" length="0.4"/>
+      </geometry>
+      <material name="Silver" />
+    </visual>
+    <collision>
+      <origin xyz="0 0 0" rpy="0 0 0" />
+      <geometry>
+        <cylinder radius="0.15" length="0.4" />
+      </geometry>
+    </collision>
+  </link>
+  <!-- Kinect vision sensor -->
+  <!-- <link name="camera_link"/>
+  <joint name="kinect_visionSensor_joint" type="fixed" >
+    <origin xyz="-0.40271 0.66297 0.796599"
+      rpy="-1.69854 -0.0579848 -2.43762"/>
+    <parent link="world_link" />
+    <child link="camera_link" />
+  </joint> -->
+  <!-- simulator-->
+  <!-- <joint name="kinect_visionSensor_joint" type="fixed" >
+    <origin xyz="-0.4568 0.6891 0.7516"
+      rpy="2.2689 0.0 1.5708"/>
+    <parent link="world_link" />
+    <child link="kinect_visionSensor" />
+  </joint> -->
 </robot>
