Commit message: a complete ping to the cartesian planner

File: ros_pkgs/hardware/lwr/lwr_description/urdf/kuka_lwr_arm_defs.xacro (robot description, xacro)
@@ -9,5 +9,5 @@
   <xacro:property name="arm_elem_end_link_mass" value="2.0"/>
   <xacro:property name="arm_elem_ball_link_mass" value="2.0"/>
-  <xacro:property name="arm_velocity_scale_factor" value="0.1"/>
+  <xacro:property name="arm_velocity_scale_factor" value="1.0"/>
   <!-- right is either 1 (for right arm) or -1 (for left arm) -->
   <xacro:macro name="kuka_lwr_arm" params="parent name right *origin">

Commit message: importing the KIT head, and supporting eddie control and planning

File: ros_pkgs/hardware/lwr/lwr_description/urdf/kuka_lwr_arm_defs.xacro (robot description, xacro)
@@ -1,7 +1,5 @@
 <?xml version="1.0"?>
-<robot xmlns:sensor="http://playerstage.sourceforge.net/gazebo/xmlschema/#sensor"
-       xmlns:controller="http://playerstage.sourceforge.net/gazebo/xmlschema/#controller"
-       xmlns:interface="http://playerstage.sourceforge.net/gazebo/xmlschema/#interface"
-       xmlns:xacro="http://www.ros.org/wiki/xacro">
+<robot xmlns:xacro="http://www.ros.org/wiki/xacro">
+  <xacro:include filename="$(find lwr_description)/urdf/materials.urdf"/>
   <xacro:include filename="$(find lwr_description)/urdf/util_defs.xacro"/>
   <xacro:property name="arm_elem_base_mass" value="2.0"/>

File: ros_pkgs/hardware/uibk_robot/urdf/uibk_robot.urdf.xacro (robot description, xacro)
@@ -1,10 +1,9 @@
 <?xml version="1.0"?>
-<robot xmlns:xacro="http://www.ros.org/wiki/xacro"
-       name="uibk_robot">
-  <xacro:include filename="$(find lwr_description)/urdf/materials.urdf"/>
+<robot xmlns:xacro="http://www.ros.org/wiki/xacro" name="Eddie">
   <xacro:include filename="$(find torso_uibk)/urdf/torso.xacro"/>
   <xacro:include filename="$(find torso_uibk)/urdf/table.xacro"/>
   <xacro:include filename="$(find lwr_description)/urdf/kuka_lwr_arm_defs.xacro"/>
   <xacro:include filename="$(find schunk_description)/urdf/sdh/sdh.urdf.xacro" />
+  <xacro:include filename="$(find kit_head_description)/model/kit_head.urdf.xacro" />
   <link name="world_link" />
   <xacro:model_table name="table"
@@ -79,25 +78,7 @@
   </xacro:schunk_sdh>
   <!-- HEAD -->
-    <!-- joint between arm_7_link and the connector ring -->
-  <joint name="world_to_kit_head" type="fixed" >
-    <origin xyz="-0.35 0.675 0.85" rpy="0 0 0" />
-    <parent link="world_link" />
-    <child link="kit_head_link" />
-  </joint>
-  <link name="kit_head_link">
-    <visual>
-      <origin xyz="0 0 0" rpy="0 0 0" />
-      <geometry>
-        <cylinder radius="0.15" length="0.4"/>
-      </geometry>
-      <material name="Silver" />
-    </visual>
-    <collision>
-      <origin xyz="0 0 0" rpy="0 0 0" />
-      <geometry>
-        <cylinder radius="0.15" length="0.4" />
-      </geometry>
-    </collision>
-  </link>
+  <xacro:kit_head name="head" parent="world">
+    <origin xyz="-0.4723 0.6767 0.85"/>
+  </xacro:kit_head>
   <!-- Kinect vision sensor -->
   <!-- <link name="camera_link"/>

Commit message: updating the cartesian planner

File: ros_pkgs/hardware/lwr/lwr_description/urdf/kuka_lwr_arm_defs.xacro (robot description, xacro)
@@ -7,5 +7,5 @@
   <xacro:property name="arm_elem_end_link_mass" value="2.0"/>
   <xacro:property name="arm_elem_ball_link_mass" value="2.0"/>
-  <xacro:property name="arm_velocity_scale_factor" value="1.0"/>
+  <xacro:property name="arm_velocity_scale_factor" value="0.1"/>
   <!-- right is either 1 (for right arm) or -1 (for left arm) -->
   <xacro:macro name="kuka_lwr_arm" params="parent name right *origin">

Commit message: improves the cart planner, first it finds a feasible cartesian path, and then it plans to generate the joint trajectory

File: ros_pkgs/hardware/lwr/lwr_description/urdf/kuka_lwr_arm_defs.xacro (robot description, xacro)
@@ -7,5 +7,5 @@
   <xacro:property name="arm_elem_end_link_mass" value="2.0"/>
   <xacro:property name="arm_elem_ball_link_mass" value="2.0"/>
-  <xacro:property name="arm_velocity_scale_factor" value="0.1"/>
+  <xacro:property name="arm_velocity_scale_factor" value="0.01"/>
   <!-- right is either 1 (for right arm) or -1 (for left arm) -->
   <xacro:macro name="kuka_lwr_arm" params="parent name right *origin">

Commit message: frame for planning fixed

File: ros_pkgs/hardware/lwr/lwr_description/urdf/kuka_lwr_arm_defs.xacro (robot description, xacro)
@@ -7,5 +7,5 @@
   <xacro:property name="arm_elem_end_link_mass" value="2.0"/>
   <xacro:property name="arm_elem_ball_link_mass" value="2.0"/>
-  <xacro:property name="arm_velocity_scale_factor" value="0.01"/>
+  <xacro:property name="arm_velocity_scale_factor" value="0.3"/>
   <!-- right is either 1 (for right arm) or -1 (for left arm) -->
   <xacro:macro name="kuka_lwr_arm" params="parent name right *origin">

Commit message: no filtering/ordering in grasp planner outputs, the grasp planners should provide an ordered list, and the trajectory planner decides whether is feasible or not to get there

File: ros_pkgs/hardware/lwr/lwr_description/urdf/kuka_lwr_arm_defs.xacro (robot description, xacro)
@@ -7,5 +7,5 @@
   <xacro:property name="arm_elem_end_link_mass" value="2.0"/>
   <xacro:property name="arm_elem_ball_link_mass" value="2.0"/>
-  <xacro:property name="arm_velocity_scale_factor" value="0.3"/>
+  <xacro:property name="arm_velocity_scale_factor" value="0.15"/>
   <!-- right is either 1 (for right arm) or -1 (for left arm) -->
   <xacro:macro name="kuka_lwr_arm" params="parent name right *origin">
