Commit message: hand joint interpolation moved to ROS.h

File: ros_pkgs/hardware/kit_head_description/model/kit_head.urdf.xacro (robot description, xacro)
@@ -149,5 +149,5 @@
         <origin xyz="0 0 0" rpy="0 0 0"/>
         <geometry>
-          <cylinder radius="0.03" length="0.03"/>
+          <cylinder radius="0.15" length="0.4"/>s
         </geometry>
       </collision>

Commit message: add bigger collision geometry for the head

File: ros_pkgs/hardware/kit_head_description/model/kit_head.urdf.xacro (robot description, xacro)
@@ -147,5 +147,5 @@
       </visual>
       <collision>
-        <origin xyz="0 0 0" rpy="0 0 0"/>
+        <origin xyz="0 0.18 0" rpy="${M_PI/2} 0 0"/>
         <geometry>
           <cylinder radius="0.15" length="0.4"/>s
